File: hardware/HackClubNano/HackClubNano.kicad_pcb (KiCad board)
At the start: 2 copper layers, 29 parts, among them J1 Conn_01x18, J2 Conn_01x02, J3 Conn_01x18, P1 USB_C_Plug_USB2.0, U1 RP2040, U2 NCP1117-3.3_SOT223, U3 W25Q128JVS, Y1 Crystal_GND24

Commit message: Finished the pcb guide. Finished the Hack Club Nano board.
Parts:
- added G***: LOGO, LOGO, B.Cu at (159.0, 92.2)
- added G***: LOGO, LOGO, B.Cu at (157.7, 114.4)
- added G***: LOGO, LOGO, B.Cu at (153.6, 84.8)
- added G***: LOGO, LOGO, B.Cu at (153.9, 104.7)
- Y1: footprint Crystal:Crystal_HC49-4H_Vertical -> Crystal:Crystal_SMD_5032-4Pin_5.0x3.2mm
- moved C14 39.9 mm to (155.4, 111.7), turned to 180 degrees
- moved U3 39.2 mm to (157.0, 115.4)
- moved J2 37.9 mm to (161.0, 81.5)
- moved C13 37.3 mm to (161.6, 111.7)
- moved R2 35.8 mm to (160.5, 88.4), turned to -90 degrees
- moved C16 34.6 mm to (151.5, 95.9), turned to 180 degrees
- moved C15 34.6 mm to (151.5, 93.1)
- moved Y1 32.6 mm to (147.6, 95.3), turned to 90 degrees
- moved C1 32.3 mm to (145.5, 81.5), turned to 90 degrees
- moved R1 31.5 mm to (157.2, 88.4), turned to -90 degrees
- moved C2 30.8 mm to (147.2, 81.5), turned to 90 degrees
- moved C7 27.0 mm to (161.6, 101.2)
- moved C8 26.5 mm to (161.6, 103.0)
- moved C9 26.0 mm to (161.6, 104.7)
- moved C10 25.5 mm to (161.6, 106.5)
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- renumbered U1 to RP2040
Routing:
- net +3.3V: track 0.00 -> 97.4 mm, vias 0 -> 11
- net Net-(J2-Pin_2): track 0.00 -> 46.2 mm, vias 0 -> 1
- net +1V1: track 0.00 -> 27.6 mm, vias 0 -> 4
- net Net-(U1-QSPI_SD0): track 0.00 -> 26.6 mm, vias 0 -> 2
- net Net-(U1-QSPI_SS): track 0.00 -> 25.2 mm, vias 0 -> 2
- net Net-(U1-QSPI_SCLK): track 0.00 -> 24.1 mm, vias 0 -> 2
- net Net-(U1-QSPI_SD2): track 0.00 -> 23.1 mm, vias 0 -> 2
- net Net-(U1-QSPI_SD3): track 0.00 -> 23.0 mm, vias 0 -> 2
- net Net-(U1-QSPI_SD1): track 0.00 -> 22.9 mm, vias 0 -> 2
- net GPIO28_ADC2: track 0.00 -> 22.3 mm, vias 0 -> 1
- net GPIO28_ADC3: track 0.00 -> 22.1 mm, vias 0 -> 1
- net GPIO0: track 0.00 -> 20.3 mm, vias 0 -> 1
- net GPIO26_ADC0: track 0.00 -> 20.1 mm, vias 0 -> 1
- net GPIO27_ADC1: track 0.00 -> 19.4 mm, vias 0 -> 1
- net GPIO1: track 0.00 -> 19.3 mm, vias 0 -> 1
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- added copper zone on In2.Cu, net GND
Other:
- board outline added: 25.4 x 43 mm
- copper layers 2 -> 4
